Commit message: Modificaciones de la clase y archivo padre

File: 2_legged_human_like_robot.urdf (robot description, URDF)
Before this commit: robot biped_robot, 7 links, 6 joints
Links:
- link base_link: geometry collision box size=0.25 0.5 0.6; visual box size=0.25 0.5 0.6
- link left_shin_link: geometry collision cylinder length=0.6 radius=0.06; visual cylinder length=0.6 radius=0.06
- link right_shin_link: geometry collision cylinder length=0.6 radius=0.06; visual cylinder length=0.6 radius=0.06
Joints:
- joint left_ankle_joint: origin xyz=0 0 0.5 rpy=0 0 0 -> xyz=0 0 -0.5 rpy=0 0 0
- joint left_hip_joint: limit lower= -0.524 upper=0.873 effort=50 velocity=2.0 -> lower= -1.0 upper=1.0 effort=50 velocity=2.0; origin xyz=0 0.25 0.05 rpy=0 0 0 -> xyz=0 0.25 -0.25 rpy=0 0 0
- joint left_knee_joint: limit lower=-1.571 upper=0 effort=50 velocity=2.0 -> lower=0 upper=1.571 effort=50 velocity=2.0; origin xyz=0 0 0.6 rpy=0 0 0 -> xyz=0 0 -0.6 rpy=0 0 0
- joint right_ankle_joint: origin xyz=0 0 0.5 rpy=0 0 0 -> xyz=0 0 -0.5 rpy=0 0 0
- joint right_hip_joint: limit lower=-0.524 upper=0.873 effort=50 velocity=2.0 -> lower=-1.0 upper=1.0 effort=50 velocity=2.0; origin xyz=0 -0.25 0.05 rpy=0 0 0 -> xyz=0 -0.25 -0.25 rpy=0 0 0
- joint right_knee_joint: limit lower=-1.571 upper=0 effort=50 velocity=2.0 -> lower=0 upper=1.571 effort=50 velocity=2.0; origin xyz=0 0 0.6 rpy=0 0 0 -> xyz=0 0 -0.6 rpy=0 0 0

Commit message: Ahora se realiza sin mover las articulaciones de tobillos

File: 2_legged_human_like_robot.urdf (robot description, URDF)
Before this commit: robot biped_robot, 7 links, 6 joints
Links:
- link base_link: geometry collision box size=0.3 0.8 0.1; visual box size=0.3 0.8 0.1
- link left_foot_link: mass 1.0 -> 1.5; geometry collision box size=0.5 0.35 0.05; visual box size=0.5 0.35 0.05
- link left_shin_link: mass 2.0 -> 4.0; geometry collision cylinder length=0.5 radius=0.06; visual cylinder length=0.5 radius=0.06
- link left_thigh_link: mass 3.0 -> 4.0
- link right_foot_link: mass 1.0 -> 1.5; geometry collision box size=0.5 0.35 0.05; visual box size=0.5 0.35 0.05
- link right_shin_link: mass 2.0 -> 4.0; geometry collision cylinder length=0.5 radius=0.06; visual cylinder length=0.5 radius=0.06
- link right_thigh_link: mass 3.0 -> 4.0
Joints:
- joint left_ankle_joint: limit lower=-0.436 upper=0.436 effort=50 velocity=2.0 -> (none); type revolute -> fixed
- joint left_hip_joint: origin xyz=0 0.25 -0.25 rpy=0 0 0 -> xyz=0 0.25 -0.05 rpy=0 0 0
- joint right_ankle_joint: limit lower=-0.436 upper=0.436 effort=50 velocity=2.0 -> (none); type revolute -> fixed
- joint right_hip_joint: origin xyz=0 -0.25 -0.25 rpy=0 0 0 -> xyz=0 -0.25 -0.05 rpy=0 0 0

Commit message: Arreglo bugs del modelo

File: 2_legged_human_like_robot.urdf (robot description, URDF)
Before this commit: robot biped_robot, 7 links, 6 joints
Links:
- link base_link: geometry collision box size=0.25 0.5 0.1; visual box size=0.25 0.5 0.1
- link left_foot_link: mass 1.0 -> 1.5
- link left_shin_link: mass 2.0 -> 4.0
- link left_thigh_link: mass 3.0 -> 4.0
- link right_foot_link: mass 1.0 -> 1.5
- link right_shin_link: mass 2.0 -> 4.0
- link right_thigh_link: mass 3.0 -> 4.0
Joints:
- joint left_hip_joint: origin xyz=0 0.25 -0.25 rpy=0 0 0 -> xyz=0 0.25 -0.0 rpy=0 0 0
- joint right_hip_joint: origin xyz=0 -0.25 -0.25 rpy=0 0 0 -> xyz=0 -0.25 -0.0 rpy=0 0 0

Commit message: Más mejoras en la visualización dle proyecto

File: 2_legged_human_like_robot.urdf (robot description, URDF)
Before this commit: robot biped_robot, 7 links, 6 joints
Links:
- link base_link: mass 8.0 -> 6.0

Commit message: Cambio de eje rotación pie

File: 2_legged_human_like_robot.urdf (robot description, URDF)
Before this commit: robot biped_robot, 7 links, 6 joints
Joints:
- joint left_ankle_joint: axis 0 1 0 -> 1 0 0; limit (none) -> lower=-0.436 upper=0.436 effort=50 velocity=2.0; type fixed -> revolute
- joint right_ankle_joint: axis 0 1 0 -> 1 0 0; limit (none) -> lower=-0.436 upper=0.436 effort=50 velocity=2.0; type fixed -> revolute

Commit message: Cambio eje rotación

File: 2_legged_human_like_robot.urdf (robot description, URDF)
Before this commit: robot biped_robot, 7 links, 6 joints
Joints:
- joint left_ankle_joint: axis 1 0 0 -> 0 1 0; limit lower=-0.436 upper=0.436 effort=50 velocity=2.0 -> lower=-0.500 upper=0.500 effort=50 velocity=2.0
- joint right_ankle_joint: axis 1 0 0 -> 0 1 0; limit lower=-0.436 upper=0.436 effort=50 velocity=2.0 -> lower=-0.500 upper=0.500 effort=50 velocity=2.0

Commit message: Realizando Arreglos en PAMIKBipedEnv

File: 2_legged_human_like_robot.urdf (robot description, URDF)
Before this commit: robot biped_robot, 7 links, 6 joints
Joints:
- joint left_hip_joint: limit lower= -1.0 upper=1.0 effort=50 velocity=2.0 -> lower= -1.2 upper=1.0 effort=50 velocity=2.0
- joint right_hip_joint: limit lower=-1.0 upper=1.0 effort=50 velocity=2.0 -> lower=-1.2 upper=1.0 effort=50 velocity=2.0

Commit message: Arreglo problema de angulos

File: 2_legged_human_like_robot.urdf (robot description, URDF)
Before this commit: robot biped_robot, 7 links, 6 joints
Joints:
- joint left_hip_joint: limit lower= -1.2 upper=1.0 effort=50 velocity=2.0 -> lower= -1.2 upper=1.2 effort=50 velocity=2.0
- joint right_hip_joint: limit lower=-1.2 upper=1.0 effort=50 velocity=2.0 -> lower=-1.2 upper=1.2 effort=50 velocity=2.0

Commit message: Modificaciones para levantar piernas

File: 2_legged_human_like_robot.urdf (robot description, URDF)
Before this commit: robot biped_robot, 7 links, 6 joints
Joints:
- joint left_ankle_joint: limit lower=-0.500 upper=0.500 effort=50 velocity=2.0 -> (none); type revolute -> fixed
- joint right_ankle_joint: limit lower=-0.500 upper=0.500 effort=50 velocity=2.0 -> (none); type revolute -> fixed

Commit message: Ligeros arreglos

File: 2_legged_human_like_robot.urdf (robot description, URDF)
Before this commit: robot biped_robot, 7 links, 6 joints
Joints:
- joint left_hip_joint: limit lower= -1.2 upper=1.2 effort=50 velocity=2.0 -> lower= -1.2 upper=0.5 effort=50 velocity=2.0
- joint right_hip_joint: limit lower=-1.2 upper=1.2 effort=50 velocity=2.0 -> lower=-1.2 upper=0.5 effort=50 velocity=2.0

Commit message: Preparaciones iniciales de co control entre caderas derecha e izquierda

File: 2_legged_human_like_robot.urdf (robot description, URDF)
Before this commit: robot biped_robot, 7 links, 6 joints
Joints:
- joint left_hip_joint: limit lower= -1.2 upper=0.5 effort=50 velocity=2.0 -> lower= -1.2 upper=1.2 effort=50 velocity=2.0
- joint right_hip_joint: limit lower=-1.2 upper=0.5 effort=50 velocity=2.0 -> lower=-1.2 upper=1.2 effort=50 velocity=2.0

Commit message: Preparación PAM 12 final

File: 2_legged_human_like_robot.urdf (robot description, URDF)
Before this commit: robot biped_robot, 7 links, 6 joints
Joints:
- joint left_ankle_joint: limit (none) -> lower=-0.500 upper=0.500 effort=50 velocity=2.0; type fixed -> revolute
- joint right_ankle_joint: limit (none) -> lower=-0.500 upper=0.500 effort=50 velocity=2.0; type fixed -> revolute
