Commit message: Modelo Preparado para 2D

File: 2_legged_human_like_robot12DOF_anckle.urdf (robot description, URDF)
Before this commit: robot biped_robot, 7 links, 6 joints
Links:
- added link right_hip_roll_link, mass 0.01
Joints:
- removed joint left_ankle_joint
- removed joint left_hip_joint
- removed joint right_ankle_joint
- removed joint right_hip_joint
- added joint left_anckle_joint: type revolute, parent left_shin_link, child left_foot_link, origin xyz=0 0 -0.5 rpy=0 0 0, axis 0 1 0, limit lower=-0.21 upper=0.21 effort=35 velocity=6.0
- added joint left_hip_pitch_joint: type revolute, parent base_link, child left_thigh_link, origin xyz=0 0.25 -0.05 rpy=0 0 0, axis 0 1 0, limit lower= -1.2 upper=1.2 effort=120 velocity=6.0
- added joint right_anckle_joint: type revolute, parent right_shin_link, child right_foot_link, origin xyz=0 0 -0.5 rpy=0 0 0, axis 0 1 0, limit lower=-0.21 upper=0.21 effort=35 velocity=6.0
- added joint right_hip_pitch_joint: type revolute, parent base_link, child right_thigh_link, origin xyz=0 -0.25 -0.05 rpy=0 0 0, axis 0 -1 0, limit lower=-1.2 upper=1.2 effort=120 velocity=6.0
