Commit message: Robot preparado para caminar

File: 2_legged_human_like_robot16DOF.urdf (robot description, URDF)
Before this commit: robot biped_robot, 9 links, 8 joints
Joints:
- joint left_knee_joint: limit lower=0 upper=1.571 effort=50 velocity=2.0 -> lower=0 upper=1.571 effort=120 velocity=6.0
- joint right_knee_joint: limit lower=0 upper=1.571 effort=50 velocity=2.0 -> lower=0 upper=1.571 effort=120 velocity=6.0
