Commit message: Robot con articulaciones listo para moverse.

File: Robots_Versiones/2_legged_human_like_robot12DOF_anckle.urdf (robot description, URDF)
Before this commit: robot biped_robot, 8 links, 6 joints
Joints:
- removed joint left_anckle_joint
- removed joint right_anckle_joint
- added joint left_ankle_joint: type revolute, parent left_shin_link, child left_foot_link, origin xyz=0 0 -0.5 rpy=0 0 0, axis 0 1 0, limit lower=-0.21 upper=0.21 effort=35 velocity=6.0
- added joint right_ankle_joint: type revolute, parent right_shin_link, child right_foot_link, origin xyz=0 0 -0.5 rpy=0 0 0, axis 0 1 0, limit lower=-0.21 upper=0.21 effort=35 velocity=6.0

File: Robots_Versiones/2_legged_human_like_robot16DOF.urdf (robot description, URDF)
Before this commit: robot biped_robot, 9 links, 8 joints
Joints:
- removed joint left_anckle_joint
- removed joint right_anckle_joint
- added joint left_ankle_joint: type revolute, parent left_shin_link, child left_foot_link, origin xyz=0 0 -0.5 rpy=0 0 0, axis 1 0 0, limit lower=-0.35 upper=0.35 effort=35 velocity=6.0
- added joint right_ankle_joint: type revolute, parent right_shin_link, child right_foot_link, origin xyz=0 0 -0.5 rpy=0 0 0, axis 1 0 0, limit lower=-0.35 upper=0.35 effort=35 velocity=6.0
- joint left_hip_roll_joint: limit lower=-0.35 upper=0.35 effort=120 velocity=6.0 -> lower=-0.25 upper=0.25 effort=120 velocity=6.0
- joint right_hip_roll_joint: limit lower=-0.35 upper=0.35 effort=120 velocity=6.0 -> lower=-0.25 upper=0.25 effort=120 velocity=6.0

File: Robots_Versiones/2_legged_human_like_robot18DOF.urdf (robot description, URDF)
Before this commit: robot biped_robot, 11 links, 10 joints
Links:
- removed link left_hip_roll_link
- removed link right_hip_roll_link
- added link left_hip_pitch_link, mass 0.05
- added link right_hip_pitch_link, mass 0.05
Joints:
- removed joint left_anckle_roll_joint
- removed joint right_anckle_roll_joint
- added joint left_ankle_roll_joint: type revolute, parent left_ankle_pitch_link, child left_foot_link, origin xyz=0 0 0.0 rpy=0 0 0, axis 1 0 0, limit lower=-0.35 upper=0.35 effort=35 velocity=6.0
- added joint right_ankle_roll_joint: type revolute, parent right_ankle_pitch_link, child right_foot_link, origin xyz=0 0 0.0 rpy=0 0 0, axis 1 0 0, limit lower=-0.35 upper=0.35 effort=35 velocity=6.0
- joint left_hip_pitch_joint: child left_thigh_link -> left_hip_pitch_link; origin xyz=0 0 0 rpy=0 0 0 -> xyz=0 0.25 -0.05 rpy=0 0 0; parent left_hip_roll_link -> base_link
- joint left_hip_roll_joint: child left_hip_roll_link -> left_thigh_link; limit lower=-0.35 upper=0.35 effort=120 velocity=6.0 -> lower=-0.25 upper=0.25 effort=120 velocity=6.0; origin xyz=0 0.25 -0.05 rpy=0 0 0 -> xyz=0 0.0 0.0 rpy=0 0 0; parent base_link -> left_hip_pitch_link
- joint right_hip_pitch_joint: child right_thigh_link -> right_hip_pitch_link; origin xyz=0 0 0 rpy=0 0 0 -> xyz=0 -0.25 -0.05 rpy=0 0 0; parent right_hip_roll_link -> base_link
- joint right_hip_roll_joint: child right_hip_roll_link -> right_thigh_link; limit lower=-0.35 upper=0.35 effort=120 velocity=6.0 -> lower=-0.25 upper=0.25 effort=120 velocity=6.0; origin xyz=0 -0.25 -0.05 rpy=0 0 0 -> xyz=0 0.0 0.0 rpy=0 0 0; parent base_link -> right_hip_pitch_link
