Commit message: Arreglo de modelo de entrenamiento 2

File: Robots_Versiones/2_legged_human_like_robot18DOF.urdf (robot description, URDF)
Before this commit: robot biped_robot, 11 links, 10 joints
Links:
- link base_link: mass 6.0 -> 5.0; geometry collision box size=0.3 0.6 0.1; visual box size=0.3 0.6 0.1
Joints:
- joint left_ankle_pitch_joint: limit lower=-0.5 upper=0.5 effort=35 velocity=6.0 -> lower=-0.5 upper=0.5 effort=60 velocity=6.0
- joint left_knee_joint: limit lower=0 upper=1.571 effort=60 velocity=6.0 -> lower=0 upper=1.571 effort=120 velocity=6.0
- joint right_ankle_pitch_joint: limit lower=-0.5 upper=0.5 effort=35 velocity=6.0 -> lower=-0.5 upper=0.5 effort=60 velocity=6.0
