Commit message: Preparando modificaciones basadas en paper

File: Robots_Versiones/2_legged_human_like_robot20DOF.urdf (robot description, URDF)
Before this commit: robot biped_robot, 11 links, 10 joints
Links:
- link left_foot_link: mass 1.5 -> 0.5; geometry collision box size=0.3 0.15 0.05; visual box size=0.3 0.15 0.05
- link right_foot_link: mass 1.5 -> 0.5; geometry collision box size=0.3 0.15 0.05; visual box size=0.3 0.15 0.05

Commit message: Elimino metodo problematico, mantengo posiciones y velocidades de COM y ZMP

File: Robots_Versiones/2_legged_human_like_robot20DOF.urdf (robot description, URDF)
Before this commit: robot biped_robot, 11 links, 10 joints
Links:
- link base_link: mass 5.0 -> 8.0

Commit message: Continuo con entrenamiento

File: Robots_Versiones/2_legged_human_like_robot20DOF.urdf (robot description, URDF)
Before this commit: robot biped_robot, 11 links, 10 joints
Links:
- link base_link: mass 8.0 -> 10.0
- link left_foot_link: geometry collision box size=0.3 0.2 0.05; visual box size=0.3 0.2 0.05
- link left_shin_link: mass 4.0 -> 3.0
- link left_thigh_link: mass 4.0 -> 3.0
- link right_foot_link: geometry collision box size=0.3 0.2 0.05; visual box size=0.3 0.2 0.05
- link right_shin_link: mass 4.0 -> 3.0
- link right_thigh_link: mass 4.0 -> 3.0

Commit message: Correccion de bugs

File: Robots_Versiones/2_legged_human_like_robot20DOF.urdf (robot description, URDF)
Before this commit: robot biped_robot, 11 links, 10 joints
Links:
- link base_link: geometry collision box size=0.3 0.6 0.2; visual box size=0.3 0.6 0.2

Commit message: Modificaciones del robot para caminar.

File: Robots_Versiones/2_legged_human_like_robot20DOF.urdf (robot description, URDF)
Before this commit: robot biped_robot, 11 links, 10 joints
Links:
- link base_link: mass 10.0 -> 12.0; geometry collision box size=0.3 0.6 0.1; visual box size=0.3 0.6 0.1
- link left_foot_link: geometry collision box size=0.4 0.3 0.05; visual box size=0.4 0.3 0.05
- link right_foot_link: geometry collision box size=0.4 0.3 0.05; visual box size=0.4 0.3 0.05

Commit message: Correcciones de roll

File: Robots_Versiones/2_legged_human_like_robot20DOF.urdf (robot description, URDF)
Before this commit: robot biped_robot, 11 links, 10 joints
Joints:
- joint left_ankle_roll_joint: limit lower=-0.35 upper=0.35 effort=35 velocity=6.0 -> lower=-0.35 upper=0.35 effort=60 velocity=6.0
- joint right_ankle_roll_joint: limit lower=-0.35 upper=0.35 effort=35 velocity=6.0 -> lower=-0.35 upper=0.35 effort=60 velocity=6.0
- joint right_knee_joint: limit lower=0 upper=1.571 effort=60 velocity=6.0 -> lower=0 upper=1.571 effort=120 velocity=6.0

Commit message: Retorno a pies anteriores

File: Robots_Versiones/2_legged_human_like_robot20DOF.urdf (robot description, URDF)
Before this commit: robot biped_robot, 11 links, 10 joints
Links:
- link left_foot_link: geometry collision box size=0.3 0.2 0.05; visual box size=0.3 0.2 0.05
- link right_foot_link: geometry collision box size=0.3 0.2 0.05; visual box size=0.3 0.2 0.05

Commit message: Retorno a masa anterior

File: Robots_Versiones/2_legged_human_like_robot20DOF.urdf (robot description, URDF)
Before this commit: robot biped_robot, 11 links, 10 joints
Links:
- link base_link: mass 12.0 -> 10.0

Commit message: Sistema que dio un paso

File: Robots_Versiones/2_legged_human_like_robot20DOF.urdf (robot description, URDF)
Before this commit: robot biped_robot, 11 links, 10 joints
Links:
- link base_link: mass 12.0 -> 10.0
Joints:
- joint left_knee_joint: limit lower=0 upper=1.571 effort=120 velocity=6.0 -> lower=0 upper=1.571 effort=60 velocity=6.0

Commit message: Preparación de nuevo modelo

File: Robots_Versiones/2_legged_human_like_robot20DOF.urdf (robot description, URDF)
Before this commit: robot biped_robot, 11 links, 10 joints
Links:
- link left_foot_link: mass 0.5 -> 0.4; geometry collision box size=0.3 0.2 0.05; visual box size=0.3 0.2 0.05
- link right_foot_link: mass 0.5 -> 0.4; geometry collision box size=0.3 0.2 0.05; visual box size=0.3 0.2 0.05

Commit message: Preparación para 20DOF

File: Robots_Versiones/2_legged_human_like_robot20DOF.urdf (robot description, URDF)
Before this commit: robot biped_robot, 11 links, 10 joints
Joints:
- joint right_hip_pitch_joint: axis 0 -1 0 -> 0 1 0
