Commit message: Reducción de caderas

File: Robots_Versiones/2_legged_human_like_robot12DOFdone_2.urdf (robot description, URDF)
Before this commit: robot biped_robot, 11 links, 10 joints
Links:
- link base_link: geometry collision box size=0.3 0.6 0.1; visual box size=0.3 0.6 0.1
- link left_shin_link: mass 2.0 -> 3.0
- link left_thigh_link: mass 2.0 -> 3.0; geometry collision cylinder length=0.6 radius=0.08; visual cylinder length=0.6 radius=0.08
- link right_shin_link: mass 2.0 -> 3.0
- link right_thigh_link: mass 2.0 -> 3.0; geometry collision cylinder length=0.6 radius=0.08; visual cylinder length=0.6 radius=0.08
Joints:
- joint left_hip_pitch_joint: origin xyz=0 0.15 -0.0 rpy=0 0 0 -> xyz=0 0.3 -0.0 rpy=0 0 0
- joint right_hip_pitch_joint: origin xyz=0 -0.15 -0.0 rpy=0 0 0 -> xyz=0 -0.3 -0.0 rpy=0 0 0
