Commit message: Modificación del robot

File: Robots_Versiones/2_legged_minihuman_legs_robot12DOF.urdf (robot description, URDF)
Before this commit: robot biped_12dof_pitch, 9 links, 8 joints
Joints:
- joint left_hip_pitch: limit lower=-0.785 upper=1.571 effort=45 velocity=8 -> lower=-0.8 upper=0.8 effort=45 velocity=8; origin xyz=0 0.08 0 rpy=0 0 0 -> xyz=0 0.08 -0.08 rpy=0 0 0
- joint right_hip_pitch: limit lower=-0.785 upper=1.571 effort=45 velocity=8 -> lower=-0.8 upper=0.8 effort=45 velocity=8; origin xyz=0 -0.08 0 rpy=0 0 0 -> xyz=0 -0.08 -0.08 rpy=0 0 0
