Commit message: Preparado para robots con distintos numeros de PAMs

File: Robots_Versiones/2_legged_human_like_robot12DOF.urdf (robot description, URDF)
Before this commit: robot biped_robot, 11 links, 10 joints
Joints:
- joint right_hip_pitch_joint: axis 0 -1 0 -> 0 1 0

File: Robots_Versiones/2_legged_human_like_robot16DOF.urdf (robot description, URDF)
Before this commit: robot biped_robot, 9 links, 8 joints
Joints:
- joint right_hip_pitch_joint: axis 0 -1 0 -> 0 1 0

File: Robots_Versiones/2_legged_human_like_robot20DOF.urdf (robot description, URDF)
Before this commit: robot biped_robot, 11 links, 10 joints
Joints:
- joint right_hip_pitch_joint: axis 0 -1 0 -> 0 1 0

Commit message: Preparando para cassie

File: Robots_Versiones/2_legged_human_like_robot12DOF.urdf (robot description, URDF)
Before this commit: robot biped_robot, 11 links, 10 joints
Joints:
- joint left_hip_pitch_joint: origin xyz=0 0.25 -0.05 rpy=0 0 0 -> xyz=0 0.3 -0.0 rpy=0 0 0
- joint right_hip_pitch_joint: origin xyz=0 -0.25 -0.05 rpy=0 0 0 -> xyz=0 -0.3 -0.0 rpy=0 0 0

Commit message: Preparando entrenamiento con minirobot

File: Robots_Versiones/2_legged_human_like_robot12DOF.urdf (robot description, URDF)
Before this commit: robot biped_robot, 11 links, 10 joints
Links:
- link base_link: geometry collision box size=0.15 0.15 0.15; visual box size=0.15 0.15 0.15
Joints:
- joint left_hip_pitch_joint: limit lower= -1.2 upper=1.2 effort=120 velocity=6.0 -> lower= -1.2 upper=1.2 effort=200 velocity=6.0; origin xyz=0 0.15 -0.0 rpy=0 0 0 -> xyz=0 0.075 0.0 rpy=0 0 0
- joint left_hip_roll_joint: limit lower=-0.25 upper=0.25 effort=120 velocity=6.0 -> lower=-0.25 upper=0.25 effort=200 velocity=6.0
- joint right_hip_pitch_joint: limit lower=-1.2 upper=1.2 effort=120 velocity=6.0 -> lower=-1.2 upper=1.2 effort=200 velocity=6.0; origin xyz=0 -0.15 -0.0 rpy=0 0 0 -> xyz=0 -0.075 -0.0 rpy=0 0 0
- joint right_hip_roll_joint: limit lower=-0.25 upper=0.25 effort=120 velocity=6.0 -> lower=-0.25 upper=0.25 effort=200 velocity=6.0
- joint right_knee_joint: limit lower=0 upper=1.571 effort=60 velocity=6.0 -> lower=0 upper=1.571 effort=200 velocity=6.0

Commit message: Preparado para aceptar robots bipedos ChatGPT

File: Robots_Versiones/2_legged_human_like_robot12DOF.urdf (robot description, URDF)
Before this commit: robot biped_robot, 11 links, 10 joints
Links:
- link base_link: geometry collision box size=0.30 0.30 0.30; visual box size=0.30 0.30 0.30
- link left_shin_link: geometry collision cylinder length=0.6 radius=0.06; visual cylinder length=0.6 radius=0.06
- link right_shin_link: geometry collision cylinder length=0.6 radius=0.06; visual cylinder length=0.6 radius=0.06
Joints:
- joint left_hip_pitch_joint: origin xyz=0 0.075 0.0 rpy=0 0 0 -> xyz=0 0.15 0.0 rpy=0 0 0
- joint right_hip_pitch_joint: origin xyz=0 -0.075 -0.0 rpy=0 0 0 -> xyz=0 -0.15 -0.0 rpy=0 0 0

File: Robots_Versiones/2_legged_minihuman_legs_robot12DOF.urdf (robot description, URDF)
Before this commit: robot biped_12dof_pitch, 9 links, 8 joints
Links:
- link pelvis: geometry collision box size=0.16 0.16 0.16; visual box size=0.16 0.16 0.16
Joints:
- joint left_hip_pitch: origin xyz=0.08 0 0 rpy=0 0 0 -> xyz=0 0.08 0 rpy=0 0 0
- joint right_hip_pitch: origin xyz=-0.08 0 0 rpy=0 0 0 -> xyz=0 -0.08 0 rpy=0 0 0

Commit message: Eliminado cancelación episodio por tilt

File: Robots_Versiones/2_legged_human_like_robot12DOF.urdf (robot description, URDF)
Before this commit: robot biped_robot, 11 links, 10 joints
Links:
- link base_link: geometry collision box size=0.30 0.30 0.30; visual box size=0.30 0.30 0.30
- link left_shin_link: geometry collision cylinder length=0.6 radius=0.06; visual cylinder length=0.6 radius=0.06
- link right_shin_link: geometry collision cylinder length=0.6 radius=0.06; visual cylinder length=0.6 radius=0.06
Joints:
- joint left_hip_pitch_joint: limit lower= -1.2 upper=1.2 effort=120 velocity=6.0 -> lower= -1.2 upper=1.2 effort=200 velocity=6.0; origin xyz=0 0.15 -0.0 rpy=0 0 0 -> xyz=0 0.15 0.0 rpy=0 0 0
- joint left_hip_roll_joint: limit lower=-0.25 upper=0.25 effort=120 velocity=6.0 -> lower=-0.25 upper=0.25 effort=200 velocity=6.0
- joint right_hip_pitch_joint: limit lower=-1.2 upper=1.2 effort=120 velocity=6.0 -> lower=-1.2 upper=1.2 effort=200 velocity=6.0
- joint right_hip_roll_joint: limit lower=-0.25 upper=0.25 effort=120 velocity=6.0 -> lower=-0.25 upper=0.25 effort=200 velocity=6.0
- joint right_knee_joint: limit lower=0 upper=1.571 effort=60 velocity=6.0 -> lower=0 upper=1.571 effort=200 velocity=6.0

Commit message: Preparación para robot con piernas de ave

File: Robots_Versiones/2_legged_human_like_robot12DOF.urdf (robot description, URDF)
Before this commit: robot biped_robot, 11 links, 10 joints
Joints:
- joint left_ankle_pitch_joint: limit lower=-0.5 upper=0.5 effort=60 velocity=6.0 -> lower=-0.6 upper=0.6 effort=60 velocity=6.0; origin xyz=0 0 -0.5 rpy=0 0 0 -> xyz=0 0 -0.6 rpy=0 0 0
- joint left_knee_joint: limit lower=0 upper=1.571 effort=60 velocity=6.0 -> lower=-1.571 upper=-0.3 effort=60 velocity=6.0
- joint right_ankle_pitch_joint: limit lower=-0.5 upper=0.5 effort=60 velocity=6.0 -> lower=-0.6 upper=0.6 effort=60 velocity=6.0; origin xyz=0 0 -0.5 rpy=0 0 0 -> xyz=0 0 -0.6 rpy=0 0 0
- joint right_knee_joint: limit lower=0 upper=1.571 effort=200 velocity=6.0 -> lower=-1.571 upper=-0.3 effort=200 velocity=6.0

Commit message: Agregadas nuevos métodos de recompensas

File: Robots_Versiones/2_legged_human_like_robot12DOF.urdf (robot description, URDF)
Before this commit: robot biped_robot, 11 links, 10 joints
Joints:
- joint left_ankle_pitch_joint: origin xyz=0 0 -0.5 rpy=0 0 0 -> xyz=0 0 -0.6 rpy=0 0 0
- joint right_ankle_pitch_joint: origin xyz=0 0 -0.5 rpy=0 0 0 -> xyz=0 0 -0.6 rpy=0 0 0

Commit message: Modifico URDF y cambio sistema

File: Robots_Versiones/2_legged_human_like_robot12DOF.urdf (robot description, URDF)
Before this commit: robot biped_robot, 11 links, 10 joints
Links:
- link left_shin_link: geometry collision cylinder length=0.4 radius=0.06; visual cylinder length=0.4 radius=0.06
- link left_thigh_link: geometry collision cylinder length=0.4 radius=0.06; visual cylinder length=0.4 radius=0.06
- link right_shin_link: geometry collision cylinder length=0.4 radius=0.06; visual cylinder length=0.4 radius=0.06
- link right_thigh_link: geometry collision cylinder length=0.4 radius=0.06; visual cylinder length=0.4 radius=0.06
Joints:
- joint left_ankle_pitch_joint: origin xyz=0 0 -0.6 rpy=0 0 0 -> xyz=0 0 -0.4 rpy=0 0 0
- joint left_knee_joint: origin xyz=0 0 -0.6 rpy=0 0 0 -> xyz=0 0 -0.4 rpy=0 0 0
- joint right_ankle_pitch_joint: origin xyz=0 0 -0.6 rpy=0 0 0 -> xyz=0 0 -0.4 rpy=0 0 0
- joint right_knee_joint: origin xyz=0 0 -0.6 rpy=0 0 0 -> xyz=0 0 -0.4 rpy=0 0 0

Commit message: Modificación de torques y castigos

File: Robots_Versiones/2_legged_human_like_robot12DOF.urdf (robot description, URDF)
Before this commit: robot biped_robot, 11 links, 10 joints
Joints:
- joint left_ankle_pitch_joint: limit lower=-0.5 upper=0.5 effort=60 velocity=6.0 -> lower=-0.5 upper=0.5 effort=60 velocity=5.0
- joint left_ankle_roll_joint: limit lower=-0.35 upper=0.35 effort=35 velocity=6.0 -> lower=-0.35 upper=0.35 effort=35 velocity=5.0
- joint left_hip_pitch_joint: limit lower= -1.2 upper=1.2 effort=200 velocity=6.0 -> lower= -1.0 upper=1.0 effort=120 velocity=6.0
- joint left_hip_roll_joint: limit lower=-0.25 upper=0.25 effort=200 velocity=6.0 -> lower=-0.25 upper=0.25 effort=120 velocity=6.0
- joint left_knee_joint: limit lower=0 upper=1.571 effort=60 velocity=6.0 -> lower=0 upper=0.9 effort=60 velocity=8.0
- joint right_ankle_pitch_joint: limit lower=-0.5 upper=0.5 effort=60 velocity=6.0 -> lower=-0.5 upper=0.5 effort=60 velocity=5.0
- joint right_ankle_roll_joint: limit lower=-0.35 upper=0.35 effort=35 velocity=6.0 -> lower=-0.35 upper=0.35 effort=35 velocity=5.0
- joint right_hip_pitch_joint: limit lower=-1.2 upper=1.2 effort=200 velocity=6.0 -> lower=-1.0 upper=1.0 effort=120 velocity=6.0
- joint right_hip_roll_joint: limit lower=-0.25 upper=0.25 effort=200 velocity=6.0 -> lower=-0.25 upper=0.25 effort=120 velocity=6.0
- joint right_knee_joint: limit lower=0 upper=1.571 effort=200 velocity=6.0 -> lower=0 upper=0.9 effort=120 velocity=8.0
