Commit message: Actualizo para llevar a main del proyecto

File: Robots_Versiones/2_legged_human_like_robot12DOF_done.urdf (robot description, URDF)
Before this commit: robot biped_robot, 11 links, 10 joints
Joints:
- joint left_ankle_pitch_joint: limit lower=-0.5 upper=0.5 effort=60 velocity=6.0 -> lower=-0.5 upper=0.5 effort=240 velocity=12.0
- joint left_ankle_roll_joint: limit lower=-0.35 upper=0.35 effort=35 velocity=6.0 -> lower=-0.35 upper=0.35 effort=240 velocity=12.0
- joint left_hip_pitch_joint: limit lower= -1.2 upper=1.2 effort=120 velocity=6.0 -> lower= -1.2 upper=1.2 effort=240 velocity=12.0
- joint left_hip_roll_joint: limit lower=-0.25 upper=0.25 effort=120 velocity=6.0 -> lower=-0.25 upper=0.25 effort=240 velocity=12.0
- joint left_knee_joint: limit lower=0 upper=1.571 effort=60 velocity=6.0 -> lower=0 upper=1.571 effort=240 velocity=12.0
- joint right_ankle_pitch_joint: limit lower=-0.5 upper=0.5 effort=60 velocity=6.0 -> lower=-0.5 upper=0.5 effort=240 velocity=12.0
- joint right_ankle_roll_joint: limit lower=-0.35 upper=0.35 effort=35 velocity=6.0 -> lower=-0.35 upper=0.35 effort=240 velocity=12.0
- joint right_hip_pitch_joint: limit lower=-1.2 upper=1.2 effort=120 velocity=6.0 -> lower=-1.2 upper=1.2 effort=240 velocity=12.0
- joint right_hip_roll_joint: limit lower=-0.25 upper=0.25 effort=120 velocity=6.0 -> lower=-0.25 upper=0.25 effort=240 velocity=12.0
- joint right_knee_joint: limit lower=0 upper=1.571 effort=60 velocity=6.0 -> lower=0 upper=1.571 effort=240 velocity=12.0
