Commit message: Modificaciones de robot y lugar de ejecución

File: Robots_Versiones/2_legged_human_like_robot16DOF.urdf (robot description, URDF)
Before this commit: robot biped_robot, 9 links, 8 joints
Joints:
- joint left_anckle_joint: limit lower=-0.21 upper=0.21 effort=35 velocity=6.0 -> lower=-0.35 upper=0.35 effort=35 velocity=6.0
- joint right_anckle_joint: limit lower=-0.21 upper=0.21 effort=35 velocity=6.0 -> lower=-0.35 upper=0.35 effort=35 velocity=6.0

Commit message: Preparación para entrenar con varios robots

File: Robots_Versiones/2_legged_human_like_robot16DOF.urdf (robot description, URDF)
Before this commit: robot biped_robot, 9 links, 8 joints
Joints:
- joint left_knee_joint: limit lower=0 upper=1.571 effort=50 velocity=2.0 -> lower=0 upper=1.571 effort=50 velocity=6.0
- joint right_knee_joint: limit lower=0 upper=1.571 effort=50 velocity=2.0 -> lower=0 upper=1.571 effort=50 velocity=6.0

File: Robots_Versiones/2_legged_human_like_robot18DOF.urdf (robot description, URDF)
Before this commit: robot biped_robot, 9 links, 8 joints
Links:
- added link left_ankle_pitch_link, mass 0.05
- added link right_ankle_pitch_link, mass 0.05
- link left_hip_roll_link: mass 0.01 -> 0.05
- link right_hip_roll_link: mass 0.01 -> 0.05
Joints:
- added joint left_ankle_pitch_joint: type revolute, parent left_shin_link, child left_ankle_pitch_link, origin xyz=0 0 -0.5 rpy=0 0 0, axis 0 1 0, limit lower=-0.5 upper=0.5 effort=35 velocity=6.0
- added joint right_ankle_pitch_joint: type revolute, parent right_shin_link, child right_ankle_pitch_link, origin xyz=0 0 -0.5 rpy=0 0 0, axis 0 1 0, limit lower=-0.5 upper=0.5 effort=35 velocity=6.0
- joint left_anckle_roll_joint: parent left_shin_link -> left_ankle_pitch_link
- joint left_knee_joint: limit lower=0 upper=1.571 effort=50 velocity=2.0 -> lower=0 upper=1.571 effort=60 velocity=6.0
- joint right_anckle_roll_joint: parent right_shin_link -> right_ankle_pitch_link
- joint right_knee_joint: limit lower=0 upper=1.571 effort=50 velocity=2.0 -> lower=0 upper=1.571 effort=60 velocity=6.0

Commit message: Arreglo de effort de rodillas

File: Robots_Versiones/2_legged_human_like_robot16DOF.urdf (robot description, URDF)
Before this commit: robot biped_robot, 9 links, 8 joints
Joints:
- joint left_knee_joint: limit lower=0 upper=1.571 effort=50 velocity=6.0 -> lower=0 upper=1.571 effort=60 velocity=6.0
- joint right_knee_joint: limit lower=0 upper=1.571 effort=50 velocity=6.0 -> lower=0 upper=1.571 effort=60 velocity=6.0

Commit message: Arreglo de modelo de entrenamiento

File: Robots_Versiones/2_legged_human_like_robot16DOF.urdf (robot description, URDF)
Before this commit: robot biped_robot, 9 links, 8 joints
Links:
- link base_link: mass 6.0 -> 5.0; geometry collision box size=0.3 0.6 0.1; visual box size=0.3 0.6 0.1
- link left_hip_roll_link: mass 0.01 -> 0.05
- link right_hip_roll_link: mass 0.01 -> 0.05

Commit message: Arreglo de modelo para entrenamiento 3

File: Robots_Versiones/2_legged_human_like_robot16DOF.urdf (robot description, URDF)
Before this commit: robot biped_robot, 9 links, 8 joints
Joints:
- removed joint left_ankle_joint
- removed joint right_ankle_joint
- added joint left_ankle_roll_joint: type revolute, parent left_shin_link, child left_foot_link, origin xyz=0 0 -0.5 rpy=0 0 0, axis 1 0 0, limit lower=-0.35 upper=0.35 effort=35 velocity=6.0
- added joint right_ankle_roll_joint: type revolute, parent right_shin_link, child right_foot_link, origin xyz=0 0 -0.5 rpy=0 0 0, axis 1 0 0, limit lower=-0.35 upper=0.35 effort=35 velocity=6.0

Commit message: Subo datos limpios

File: Robots_Versiones/2_legged_human_like_robot16DOF.urdf (robot description, URDF)
Before this commit: robot biped_robot, 9 links, 8 joints
Links:
- removed link left_hip_roll_link
- removed link right_hip_roll_link
- added link left_ankle_pitch_link, mass 0.05
- added link left_hip_pitch_link, mass 0.05
- added link right_ankle_pitch_link, mass 0.05
- added link right_hip_pitch_link, mass 0.05
- link base_link: mass 5.0 -> 10.0
- link left_foot_link: mass 1.5 -> 0.4; geometry collision box size=0.3 0.2 0.05; visual box size=0.3 0.2 0.05
- link left_shin_link: mass 4.0 -> 3.0
- link left_thigh_link: mass 4.0 -> 3.0
- link right_foot_link: mass 1.5 -> 0.4; geometry collision box size=0.3 0.2 0.05; visual box size=0.3 0.2 0.05
- link right_shin_link: mass 4.0 -> 3.0
- link right_thigh_link: mass 4.0 -> 3.0
Joints:
- added joint left_ankle_pitch_joint: type revolute, parent left_shin_link, child left_ankle_pitch_link, origin xyz=0 0 -0.5 rpy=0 0 0, axis 0 1 0, limit lower=-0.5 upper=0.5 effort=240 velocity=12.0
- added joint right_ankle_pitch_joint: type revolute, parent right_shin_link, child right_ankle_pitch_link, origin xyz=0 0 -0.5 rpy=0 0 0, axis 0 1 0, limit lower=-0.5 upper=0.5 effort=240 velocity=12.0
- joint left_ankle_roll_joint: limit lower=-0.35 upper=0.35 effort=35 velocity=6.0 -> lower=-0.35 upper=0.35 effort=240 velocity=12.0; origin xyz=0 0 -0.5 rpy=0 0 0 -> xyz=0 0 0.0 rpy=0 0 0; parent left_shin_link -> left_ankle_pitch_link; type revolute -> fixed
- joint left_hip_pitch_joint: child left_thigh_link -> left_hip_pitch_link; limit lower= -1.2 upper=1.2 effort=120 velocity=6.0 -> lower= -1.2 upper=1.2 effort=240 velocity=12.0; origin xyz=0 0 0 rpy=0 0 0 -> xyz=0 0.25 -0.05 rpy=0 0 0; parent left_hip_roll_link -> base_link
- joint left_hip_roll_joint: child left_hip_roll_link -> left_thigh_link; limit lower=-0.25 upper=0.25 effort=120 velocity=6.0 -> lower=-0.25 upper=0.25 effort=240 velocity=12.0; origin xyz=0 0.25 -0.05 rpy=0 0 0 -> xyz=0 0.0 0.0 rpy=0 0 0; parent base_link -> left_hip_pitch_link
- joint left_knee_joint: limit lower=0 upper=1.571 effort=60 velocity=6.0 -> lower=0 upper=1.571 effort=240 velocity=12.0
- joint right_ankle_roll_joint: limit lower=-0.35 upper=0.35 effort=35 velocity=6.0 -> lower=-0.35 upper=0.35 effort=240 velocity=12.0; origin xyz=0 0 -0.5 rpy=0 0 0 -> xyz=0 0 0.0 rpy=0 0 0; parent right_shin_link -> right_ankle_pitch_link; type revolute -> fixed
- joint right_hip_pitch_joint: child right_thigh_link -> right_hip_pitch_link; limit lower=-1.2 upper=1.2 effort=120 velocity=6.0 -> lower=-1.2 upper=1.2 effort=240 velocity=12.0; origin xyz=0 0 0 rpy=0 0 0 -> xyz=0 -0.25 -0.05 rpy=0 0 0; parent right_hip_roll_link -> base_link
- joint right_hip_roll_joint: child right_hip_roll_link -> right_thigh_link; limit lower=-0.25 upper=0.25 effort=120 velocity=6.0 -> lower=-0.25 upper=0.25 effort=240 velocity=12.0; origin xyz=0 -0.25 -0.05 rpy=0 0 0 -> xyz=0 0.0 0.0 rpy=0 0 0; parent base_link -> right_hip_pitch_link
- joint right_knee_joint: limit lower=0 upper=1.571 effort=60 velocity=6.0 -> lower=0 upper=1.571 effort=240 velocity=12.0

File: Robots_Versiones/2_legged_human_like_robot20DOF.urdf (robot description, URDF)
Before this commit: robot biped_robot, 11 links, 10 joints
Joints:
- joint left_ankle_pitch_joint: limit lower=-0.5 upper=0.5 effort=60 velocity=6.0 -> lower=-0.5 upper=0.5 effort=240 velocity=12.0
- joint left_ankle_roll_joint: limit lower=-0.35 upper=0.35 effort=35 velocity=6.0 -> lower=-0.35 upper=0.35 effort=240 velocity=12.0
- joint left_hip_pitch_joint: limit lower= -1.2 upper=1.2 effort=120 velocity=6.0 -> lower= -1.2 upper=1.2 effort=240 velocity=12.0
- joint left_hip_roll_joint: limit lower=-0.25 upper=0.25 effort=120 velocity=6.0 -> lower=-0.25 upper=0.25 effort=240 velocity=12.0
- joint left_knee_joint: limit lower=0 upper=1.571 effort=60 velocity=6.0 -> lower=0 upper=1.571 effort=240 velocity=12.0
- joint right_ankle_pitch_joint: limit lower=-0.5 upper=0.5 effort=60 velocity=6.0 -> lower=-0.5 upper=0.5 effort=240 velocity=12.0
- joint right_ankle_roll_joint: limit lower=-0.35 upper=0.35 effort=35 velocity=6.0 -> lower=-0.35 upper=0.35 effort=240 velocity=12.0
- joint right_hip_pitch_joint: limit lower=-1.2 upper=1.2 effort=120 velocity=6.0 -> lower=-1.2 upper=1.2 effort=240 velocity=12.0
- joint right_hip_roll_joint: limit lower=-0.25 upper=0.25 effort=120 velocity=6.0 -> lower=-0.25 upper=0.25 effort=240 velocity=12.0
- joint right_knee_joint: limit lower=0 upper=1.571 effort=60 velocity=6.0 -> lower=0 upper=1.571 effort=240 velocity=12.0
