Commit message: Adaptación torques

File: Robots_Versiones/Robots_Rodilla_Invertida/2_legged_human_like_robotInverse_knees_12DOF.urdf (robot description, URDF)
Before this commit: robot biped_robot, 11 links, 10 joints
Joints:
- joint left_knee_joint: limit lower=-1.571 upper=0 effort=60 velocity=6.0 -> lower=-1.571 upper=-0.2 effort=60 velocity=6.0
- joint right_knee_joint: limit lower=-1.571 upper=0 effort=60 velocity=6.0 -> lower=-1.571 upper=-0.2 effort=60 velocity=6.0
