Commit message: Adaptado para blackbird

File: Robots_Versiones/Black_bird/urdf/blackbird.urdf (robot description, URDF)
Before this commit: robot biped, 11 links, 10 joints
Joints:
- joint l_ab_ad: limit lower=-2 upper=2 effort=0 velocity=0 -> lower=-2 upper=2 effort=100 velocity=6
- joint l_foot: limit lower=-1.5708 upper=0.69813 effort=0 velocity=0 -> lower=-1.5708 upper=0.69813 effort=30 velocity=4
- joint l_lower: limit lower=-2.0944 upper=0.34907 effort=0 velocity=0 -> lower=-2.0944 upper=0.34907 effort=40 velocity=4
- joint l_upper: limit lower=-1.91986 upper=1.22173 effort=0 velocity=0 -> lower=-1.91986 upper=1.22173 effort=80 velocity=5
- joint l_yaw: limit lower=-2 upper=2 effort=0 velocity=0 -> lower=-2 upper=2 effort=100 velocity=6
- joint r_ab_ad: limit lower=-2 upper=2 effort=0 velocity=0 -> lower=-2 upper=2 effort=100 velocity=6
- joint r_foot: limit lower=-1.5708 upper=0.69813 effort=0 velocity=0 -> lower=-1.5708 upper=0.69813 effort=30 velocity=4
- joint r_lower: limit lower=-2.0944 upper=0.34907 effort=0 velocity=0 -> lower=-2.0944 upper=0.34907 effort=40 velocity=4
- joint r_upper: limit lower=-1.91986 upper=1.22173 effort=0 velocity=0 -> lower=-1.91986 upper=1.22173 effort=80 velocity=5
- joint r_yaw: limit lower=-2 upper=2 effort=0 velocity=0 -> lower=-2 upper=2 effort=100 velocity=6
